File: PowerControl_PCM_V0.1_Power/PowerControl_PCM_V0.1_Power.kicad_pcb (KiCad board)
At the start: 2 copper layers, 44 x 60 mm, 74 parts, among them J12 Conn_M, J13 Conn_M, J14 Conn_M, J15 Conn_M, J16 Conn_M, J2 XT30-F, J3 Conn_M, J4 XT30-M, J5 XT30-M, J6 XT30-M, J7 Conn_M, Q1 BSC070N10N, Q2 BSC070N10N, Q3 BSC070N10N, Q4 BSC070N10N, Q5 BSC070N10N, Q6 BSC070N10N, U1 UCC27201A, U2 UCC27211, U3 UCC27211

Commit message: 修复电容旋转问题
Parts:
- turned C1 to 180 degrees
